File: Banshee/Banshee.sch (KiCad schematic (older format))
At the start: 24 parts, among them J1 4mmPad, J2 4mmPad, J3 Conn_01x03_Male, J4 4mmPad, J5 4mmPad, J6 4mmPad, J7 4mmPad, U1 ESP32-DEVKITC-32D, U2 AMS1117, U3 L293D

Commit message: minor electrical design edits
Parts:
- removed C1, C2: 10u, Capacitor_THT:CP_Radial_D5.0mm_P2.50mm, symbol Device:C
- removed D1, D2, D3, D4, D5, D6, D8: 1N4002, Diode_THT:D_A-405_P12.70mm_Horizontal, symbol Device:D
- removed H1, H2, H3, H4: MountingHole, MountingHole:MountingHole_3.2mm_M3_Pad, symbol Mechanical:MountingHole
- removed J1, J2, J4, J5, J6, J7: 4mmPad, customFootprints:4mmPad, symbol customParts:4mmPad
- added C?: 470u, symbol Device:CP1
- added J? (x4): Conn_01x02_Female, symbol Connector:Conn_01x02_Female
Connections:
- net +5V: now also C?.1; no longer D7.1 (K)
- net GND: now also C?.2, J?.1 (Pin_1), J?.1 (Pin_1)
- net M1+: now also J?.2 (Pin_2)
- net M1-: now also J?.1 (Pin_1)
- net M2+: now also J?.2 (Pin_2)
- net M2-: now also J?.1 (Pin_1); no longer D7.2 (A)
- net Motor_1A: now also U1.31 (IO16); no longer U1.32 (IO4)
- net Motor_2A: now also U1.32 (IO4); no longer U1.31 (IO16)
- net Motor_2EN: now also U1.10 (IO26); no longer U1.12 (IO14)
- net Motor_3A: now also U1.11 (IO27); no longer U1.10 (IO26)
- net Motor_4A: now also U1.12 (IO14); no longer U1.11 (IO27)
- net at U2.3 (VI): now also D7.1 (K)
- new net Bat+: D7.2 (A), J?.2 (Pin_2), J?.2 (Pin_2)
Other:
- note added: "*XT30U connectors\n"
- note removed: "Mounting"
- moved on the sheet: D7

Commit message: added simple voltage divider to sense battery voltage
Parts:
- added H1, H2, H3, H4: MountingHole, MountingHole:MountingHole_3.2mm_M3_Pad, symbol Mechanical:MountingHole
- added R?: 22k, symbol Device:R
- added R?: 2.2k, symbol Device:R
Connections:
- net labels added: BAT_SENSE
- wire segments 50 -> 55
Other:
- note added: "Mounting"
Changed lines of the file:
@@
 Wire Notes Line
 	6450 3600 4100 3600
+$Comp
+L Mechanical:MountingHole H1
+U 1 1 60575BBE
+P 6000 6550
+F 0 "H1" H 6100 6596 50  0000 L CNN
+F 1 "MountingHole" H 6100 6505 50  0000 L CNN
+F 2 "MountingHole:MountingHole_3.2mm_M3_Pad" H 6000 6550 50  0001 C CNN
+F 3 "~" H 6000 6550 50  0001 C CNN
+	1    6000 6550
+	1    0    0    -1
+$EndComp
+$Comp
+L Mechanical:MountingHole H2
+U 1 1 60577AD4
+P 6000 6850
+F 0 "H2" H 6100 6896 50  0000 L CNN
+F 1 "MountingHole" H 6100 6805 50  0000 L CNN
+F 2 "MountingHole:MountingHole_3.2mm_M3_Pad" H 6000 6850 50  0001 C CNN
+F 3 "~" H 6000 6850 50  0001 C CNN
+	1    6000 6850
+	1    0    0    -1
+$EndComp
+$Comp
+L Mechanical:MountingHole H3
+U 1 1 60577E22
+P 6000 7150
+F 0 "H3" H 6100 7196 50  0000 L CNN
+F 1 "MountingHole" H 6100 7105 50  0000 L CNN
+F 2 "MountingHole:MountingHole_3.2mm_M3_Pad" H 6000 7150 50  0001 C CNN
+F 3 "~" H 6000 7150 50  0001 C CNN
+	1    6000 7150
+	1    0    0    -1
+$EndComp
+$Comp
+L Mechanical:MountingHole H4
+U 1 1 60578051
+P 6000 7450
+F 0 "H4" H 6100 7496 50  0000 L CNN
+F 1 "MountingHole" H 6100 7405 50  0000 L CNN
+F 2 "MountingHole:MountingHole_3.2mm_M3_Pad" H 6000 7450 50  0001 C CNN
+F 3 "~" H 6000 7450 50  0001 C CNN
+	1    6000 7450
+	1    0    0    -1
+$EndComp
 Text Notes 700  2550 0    50   ~ 0
 ESP32
+Text Notes 5850 6400 0    50   ~ 0
+Mounting
+Wire Notes Line
+	5800 6300 5800 7750
+Wire Notes Line
+	5800 7750 6900 7750
+Wire Notes Line
+	6900 7750 6900 6300
+Wire Notes Line
+	5800 6300 6900 6300
 Wire Wire Line
 	1050 1000 1350 1000
@@
 Wire Wire Line
 	1200 1100 1200 1200
-Text Label 1100 1000 0    50   ~ 0
+Text Label 1150 1000 0    50   ~ 0
 Bat+
 $Comp
@@
 	1    0    0    -1
 $EndComp
+$Comp
+L Device:R R?
+U 1 1 604C396B
+P 4700 5400
+F 0 "R?" H 4770 5446 50  0000 L CNN
+F 1 "22k" H 4770 5355 50  0000 L CNN
+F 2 "" V 4630 5400 50  0001 C CNN
+F 3 "~" H 4700 5400 50  0001 C CNN
+	1    4700 5400
+	1    0    0    -1
+$EndComp
+$Comp
+L Device:R R?
+U 1 1 604C42A2
+P 4700 5900
+F 0 "R?" H 4770 5946 50  0000 L CNN
+F 1 "2.2k" H 4770 5855 50  0000 L CNN
+F 2 "" V 4630 5900 50  0001 C CNN
+F 3 "~" H 4700 5900 50  0001 C CNN
+	1    4700 5900
+	1    0    0    -1
+$EndComp
+Text Label 4850 5100 0    50   ~ 0
+Bat+
+Wire Wire Line
+	4850 5100 4700 5100
+Wire Wire Line
+	4700 5100 4700 5250
+Wire Wire Line
+	4700 5550 4700 5750
+$Comp
+L power:GND #PWR?
+U 1 1 604C94FF
+P 4700 6250
+F 0 "#PWR?" H 4700 6000 50  0001 C CNN
+F 1 "GND" H 4705 6077 50  0000 C CNN
+F 2 "" H 4700 6250 50  0001 C CNN
+F 3 "" H 4700 6250 50  0001 C CNN
+	1    4700 6250
+	1    0    0    -1
+$EndComp
+Wire Wire Line
+	4700 6250 4700 6050
+Text Label 5200 5650 2    50   ~ 0
+BAT_SENSE
+Text Label 3650 6100 2    50   ~ 0
+BAT_SENSE
+Wire Wire Line
+	3650 6100 3050 6100
 $EndSCHEMATC
