File: Electrical/Banshee.sch (KiCad schematic (older format))
At the start: 16 parts, among them J3 Conn_01x03_Male, U1 ESP32-DEVKITC-32D, U2 AMS1117, U3 L293D

Commit message: minior schematic edits
Parts:
- removed H1, H2, H3, H4: MountingHole, MountingHole:MountingHole_3.2mm_M3_Pad, symbol Mechanical:MountingHole
Connections:
- wire segments 55 -> 57
Other:
- note added: "Battery Sense"
- note removed: "Mounting"
- moved on the sheet: R?
Changed lines of the file:
@@
 Wire Notes Line
 	6450 3600 4100 3600
-$Comp
-L Mechanical:MountingHole H1
-U 1 1 60575BBE
-P 6000 6550
-F 0 "H1" H 6100 6596 50  0000 L CNN
-F 1 "MountingHole" H 6100 6505 50  0000 L CNN
-F 2 "MountingHole:MountingHole_3.2mm_M3_Pad" H 6000 6550 50  0001 C CNN
-F 3 "~" H 6000 6550 50  0001 C CNN
-	1    6000 6550
-	1    0    0    -1
-$EndComp
-$Comp
-L Mechanical:MountingHole H2
-U 1 1 60577AD4
-P 6000 6850
-F 0 "H2" H 6100 6896 50  0000 L CNN
-F 1 "MountingHole" H 6100 6805 50  0000 L CNN
-F 2 "MountingHole:MountingHole_3.2mm_M3_Pad" H 6000 6850 50  0001 C CNN
-F 3 "~" H 6000 6850 50  0001 C CNN
-	1    6000 6850
-	1    0    0    -1
-$EndComp
-$Comp
-L Mechanical:MountingHole H3
-U 1 1 60577E22
-P 6000 7150
-F 0 "H3" H 6100 7196 50  0000 L CNN
-F 1 "MountingHole" H 6100 7105 50  0000 L CNN
-F 2 "MountingHole:MountingHole_3.2mm_M3_Pad" H 6000 7150 50  0001 C CNN
-F 3 "~" H 6000 7150 50  0001 C CNN
-	1    6000 7150
-	1    0    0    -1
-$EndComp
-$Comp
-L Mechanical:MountingHole H4
-U 1 1 60578051
-P 6000 7450
-F 0 "H4" H 6100 7496 50  0000 L CNN
-F 1 "MountingHole" H 6100 7405 50  0000 L CNN
-F 2 "MountingHole:MountingHole_3.2mm_M3_Pad" H 6000 7450 50  0001 C CNN
-F 3 "~" H 6000 7450 50  0001 C CNN
-	1    6000 7450
-	1    0    0    -1
-$EndComp
 Text Notes 700  2550 0    50   ~ 0
 ESP32
-Text Notes 5850 6400 0    50   ~ 0
-Mounting
-Wire Notes Line
-	5800 6300 5800 7750
-Wire Notes Line
-	5800 7750 6900 7750
-Wire Notes Line
-	6900 7750 6900 6300
-Wire Notes Line
-	5800 6300 6900 6300
 Wire Wire Line
 	1050 1000 1350 1000
@@
 L Device:R R?
 U 1 1 604C396B
-P 4700 5400
-F 0 "R?" H 4770 5446 50  0000 L CNN
-F 1 "22k" H 4770 5355 50  0000 L CNN
-F 2 "" V 4630 5400 50  0001 C CNN
-F 3 "~" H 4700 5400 50  0001 C CNN
-	1    4700 5400
+P 5200 5400
+F 0 "R?" H 5270 5446 50  0000 L CNN
+F 1 "22k" H 5270 5355 50  0000 L CNN
+F 2 "" V 5130 5400 50  0001 C CNN
+F 3 "~" H 5200 5400 50  0001 C CNN
+	1    5200 5400
 	1    0    0    -1
 $EndComp
@@
 L Device:R R?
 U 1 1 604C42A2
-P 4700 5900
-F 0 "R?" H 4770 5946 50  0000 L CNN
-F 1 "2.2k" H 4770 5855 50  0000 L CNN
-F 2 "" V 4630 5900 50  0001 C CNN
-F 3 "~" H 4700 5900 50  0001 C CNN
-	1    4700 5900
+P 5200 5900
+F 0 "R?" H 5270 5946 50  0000 L CNN
+F 1 "2.2k" H 5270 5855 50  0000 L CNN
+F 2 "" V 5130 5900 50  0001 C CNN
+F 3 "~" H 5200 5900 50  0001 C CNN
+	1    5200 5900
 	1    0    0    -1
 $EndComp
-Text Label 4850 5100 0    50   ~ 0
+Text Label 5350 5100 0    50   ~ 0
 Bat+
 Wire Wire Line
-	4850 5100 4700 5100
+	5350 5100 5200 5100
 Wire Wire Line
-	4700 5100 4700 5250
+	5200 5100 5200 5250
 Wire Wire Line
-	4700 5550 4700 5750
+	5200 5550 5200 5650
 $Comp
 L power:GND #PWR?
 U 1 1 604C94FF
-P 4700 6250
-F 0 "#PWR?" H 4700 6000 50  0001 C CNN
-F 1 "GND" H 4705 6077 50  0000 C CNN
-F 2 "" H 4700 6250 50  0001 C CNN
-F 3 "" H 4700 6250 50  0001 C CNN
-	1    4700 6250
+P 5200 6250
+F 0 "#PWR?" H 5200 6000 50  0001 C CNN
+F 1 "GND" H 5205 6077 50  0000 C CNN
+F 2 "" H 5200 6250 50  0001 C CNN
+F 3 "" H 5200 6250 50  0001 C CNN
+	1    5200 6250
 	1    0    0    -1
 $EndComp
 Wire Wire Line
-	4700 6250 4700 6050
-Text Label 5200 5650 2    50   ~ 0
+	5200 6250 5200 6050
+Text Label 5700 5650 2    50   ~ 0
 BAT_SENSE
 Text Label 3650 6100 2    50   ~ 0
@@
 Wire Wire Line
 	3650 6100 3050 6100
+Wire Wire Line
+	5700 5650 5200 5650
+Connection ~ 5200 5650
+Wire Wire Line
+	5200 5650 5200 5750
+Wire Notes Line
+	4100 4900 6450 4900
+Wire Notes Line
+	6450 4900 6450 6600
+Wire Notes Line
+	6450 6600 4100 6600
+Wire Notes Line
+	4100 6600 4100 4900
+Text Notes 4150 5050 0    50   ~ 0
+Battery Sense
 $EndSCHEMATC
